Commit message: feat: add Robotiq 3F gripper

File: src/arm_description/urdf/ros2_control_gz.xacro (robot description, xacro)
@@ -3,7 +3,22 @@
   <xacro:include filename="$(find arm_description)/urdf/inc/ur_joint_control.xacro" />
   <xacro:include filename="$(find arm_description)/urdf/inc/ur_sensors.xacro" />
+  <xacro:macro name="gz_position_controlled_joint" params="joint_name">
+    <joint name="${joint_name}">
+      <command_interface name="position"/>
+      <state_interface name="position">
+        <param name="initial_value">0.0</param>
+      </state_interface>
+      <state_interface name="velocity">
+        <param name="initial_value">0.0</param>
+      </state_interface>
+      <state_interface name="effort">
+        <param name="initial_value">0.0</param>
+      </state_interface>
+    </joint>
+  </xacro:macro>
   <xacro:macro name="ur_gz_ros2_control" params="
     name
     tf_prefix
+    gripper_prefix:=robotiq_
     initial_positions:=${dict(shoulder_pan_joint=0.0,shoulder_lift_joint=-1.57,elbow_joint=0.0,wrist_1_joint=-1.57,wrist_2_joint=0.0,wrist_3_joint=0.0)}
     ">
@@ -19,4 +34,15 @@
         tf_prefix="${tf_prefix}"
       />
+      <xacro:gz_position_controlled_joint joint_name="${tf_prefix}${gripper_prefix}palm_finger_1_joint"/>
+      <xacro:gz_position_controlled_joint joint_name="${tf_prefix}${gripper_prefix}finger_1_joint_1"/>
+      <xacro:gz_position_controlled_joint joint_name="${tf_prefix}${gripper_prefix}finger_1_joint_2"/>
+      <xacro:gz_position_controlled_joint joint_name="${tf_prefix}${gripper_prefix}finger_1_joint_3"/>
+      <xacro:gz_position_controlled_joint joint_name="${tf_prefix}${gripper_prefix}palm_finger_2_joint"/>
+      <xacro:gz_position_controlled_joint joint_name="${tf_prefix}${gripper_prefix}finger_2_joint_1"/>
+      <xacro:gz_position_controlled_joint joint_name="${tf_prefix}${gripper_prefix}finger_2_joint_2"/>
+      <xacro:gz_position_controlled_joint joint_name="${tf_prefix}${gripper_prefix}finger_2_joint_3"/>
+      <xacro:gz_position_controlled_joint joint_name="${tf_prefix}${gripper_prefix}finger_middle_joint_1"/>
+      <xacro:gz_position_controlled_joint joint_name="${tf_prefix}${gripper_prefix}finger_middle_joint_2"/>
+      <xacro:gz_position_controlled_joint joint_name="${tf_prefix}${gripper_prefix}finger_middle_joint_3"/>
     </ros2_control>
   </xacro:macro>

File: src/arm_description/urdf/ur.urdf.xacro (robot description, xacro)
@@ -5,4 +5,6 @@
    <!-- import main macro -->
    <xacro:include filename="$(find arm_description)/urdf/ur_macro.xacro"/>
+   <xacro:include filename="$(find arm_description)/urdf/robotiq_3f_mount.xacro" />
+   <xacro:include filename="$(find arm_description)/urdf/realsense_d435i_mount.xacro" />
    <!-- possible 'ur_type' values: ur3, ur5, ur10, ur3e, ur5e, ur7e, ur10e, ur12e, ur16e, ur8long, ur15, ur18, ur20, ur30 -->
    <!-- the default value should raise an error in case this was called without defining the type -->
@@ -20,4 +22,5 @@
    <!--When using gazebo simulations absolute paths are necessary.-->
    <xacro:arg name="force_abs_paths" default="false" />
+   <xacro:arg name="gripper_prefix" default="robotiq_"/>
    <!-- create link fixed to the "world" -->
    <link name="world" />
@@ -38,3 +41,9 @@
      <origin xyz="0 0 0" rpy="0 0 0" />          <!-- position robot in the world -->
    </xacro:ur_robot>
+   <xacro:robotiq_3f_mount parent="$(arg tf_prefix)tool0" prefix="$(arg tf_prefix)$(arg gripper_prefix)">
+     <origin xyz="0 0 0.045" rpy="1.5708 0 0"/>
+   </xacro:robotiq_3f_mount>
+   <xacro:realsense_d435i_mount parent="$(arg tf_prefix)$(arg gripper_prefix)palm" name="$(arg tf_prefix)wrist_camera">
+     <origin xyz="0 0 0.095" rpy="0 ${-pi/2} 0"/>
+   </xacro:realsense_d435i_mount>
 </robot>

File: src/arm_description/urdf/ur_gz_controlled.urdf.xacro (robot description, xacro)
@@ -4,4 +4,6 @@
   <xacro:include filename="$(find arm_description)/urdf/ur_macro.xacro"/>
   <xacro:include filename="$(find arm_description)/urdf/ros2_control_gz.xacro" />
+  <xacro:include filename="$(find arm_description)/urdf/robotiq_3f_mount.xacro" />
+  <xacro:include filename="$(find arm_description)/urdf/realsense_d435i_mount.xacro" />
   <xacro:arg name="ur_type" default="ur5e"/>
   <xacro:arg name="tf_prefix" default="" />
@@ -16,4 +18,5 @@
   <xacro:arg name="initial_positions_file" default="$(find arm_description)/config/initial_positions.yaml"/>
   <xacro:arg name="controllers_file" default="$(find arm_ros2_control)/config/controllers.yaml"/>
+  <xacro:arg name="gripper_prefix" default="robotiq_"/>
   <xacro:property name="initial_positions_file" default="$(arg initial_positions_file)"/>
   <link name="world" />
@@ -33,7 +36,14 @@
     <origin xyz="0 0 0" rpy="0 0 0" />
   </xacro:ur_robot>
+  <xacro:robotiq_3f_mount parent="$(arg tf_prefix)tool0" prefix="$(arg tf_prefix)$(arg gripper_prefix)">
+    <origin xyz="0 0 0.045" rpy="1.5708 0 0"/>
+  </xacro:robotiq_3f_mount>
+  <xacro:realsense_d435i_mount parent="$(arg tf_prefix)$(arg gripper_prefix)palm" name="$(arg tf_prefix)wrist_camera">
+    <origin xyz="0 0 0.095" rpy="0 ${-pi/2} 0"/>
+  </xacro:realsense_d435i_mount>
   <xacro:ur_gz_ros2_control
     name="$(arg name)"
     tf_prefix="$(arg tf_prefix)"
+    gripper_prefix="$(arg gripper_prefix)"
     initial_positions="${xacro.load_yaml(initial_positions_file)}"
   />
